Commit message: Teleoperate rover in gazebo

File: zeus_description/urdf/zeus.urdf.xacro (robot description, xacro)
@@ -18,9 +18,6 @@
   <xacro:property name="wheel_kp" value="10000000.0" />
   <xacro:property name="wheel_kd" value="1" />
-  <!-- High level dummy link for ODE -->
+  <!-- Frame -->
   <link name="base_link">
-  </link>
-  <!-- Frame -->
-  <link name="frame_link">
     <visual>
       <geometry>
@@ -33,5 +30,5 @@
         <box size="${frame_length} ${frame_width} ${frame_height}"/>
       </geometry>
-      <origin rpy="0 0 0" xyz="-0.27 -0.02 -0.45"/>
+      <origin rpy="0 0 0" xyz="0 0 0"/>
     </collision>
     <inertial>
@@ -40,11 +37,6 @@
     </inertial>
   </link>
-  <joint name="frame_link_joint" type="fixed">
-    <parent link="base_link"/>
-    <child link="frame_link"/>
-    <origin rpy="0 -0 0" xyz="0 0 0"/>
-  </joint>
-  <gazebo reference="frame_link">
-    <material>Gazebo/DarkGray</material>
+  <gazebo reference="base_link">
+    <!-- <material>Gazebo/DarkGray</material> -->
   </gazebo>
 <!-- Rocker right -->
@@ -62,5 +54,5 @@
   </link>
   <joint name="rocker_right_joint" type="revolute">
-    <parent link="frame_link"/>
+    <parent link="base_link"/>
     <child link="rocker_right"/>
     <origin rpy="0 -0.2 0" xyz="-0.3 -0.3 -0.4"/>
@@ -80,5 +72,5 @@
   </transmission>
   <gazebo reference="rocker_right">
-    <material>Gazebo/Gray</material>
+    <!-- <material>Gazebo/Gray</material> -->
   </gazebo>
   <!-- Bogie right -->
@@ -89,5 +81,5 @@
       </geometry>
       <origin rpy="0 0 0" xyz="0 0 0"/>
-      <material name="gray"/>
+      <!-- <material name="gray"/> -->
     </visual>
     <inertial>
@@ -105,5 +97,5 @@
   </joint>
   <gazebo reference="bogie_right">
-    <material>Gazebo/Gray</material>
+    <!-- <material>Gazebo/Gray</material> -->
   </gazebo>
   <!-- Rocker left -->
@@ -114,5 +106,5 @@
       </geometry>
       <origin rpy="0 0 0" xyz="0 0 0"/>
-      <material name="gray"/>
+      <!-- <material name="gray"/> -->
     </visual>
     <inertial>
@@ -121,6 +113,6 @@
     </inertial>
   </link>
-  <joint name="rocker_left_joint" type="continuous">
-    <parent link="frame_link"/>
+  <joint name="rocker_left_joint" type="revolute">
+    <parent link="base_link"/>
     <child link="rocker_left"/>
     <origin rpy="0 -0.2 0" xyz="-0.3 0.3 -0.4"/>
@@ -140,6 +132,6 @@
   </transmission>
   <gazebo reference="rocker_left">
-    <material>Gazebo/Gray</material>
-  </gazebo>
+    <!-- <material>Gazebo/Gray</material> -->
+  </gazebo> -->
   <!-- Bogie left -->
   <link name="bogie_left">
@@ -149,5 +141,5 @@
       </geometry>
       <origin rpy="0 0 0" xyz="0 0 0"/>
-      <material name="gray"/>
+      <!-- <material name="gray"/> -->
     </visual>
     <inertial>
@@ -165,5 +157,5 @@
   </joint>
   <gazebo reference="bogie_left">
-    <material>Gazebo/Gray</material>
+    <!-- <material>Gazebo/Gray</material> -->
   </gazebo>
   <!-- Wheel front right -->
@@ -207,5 +199,5 @@
     <kp value="${wheel_kp}" />
     <kd value="${wheel_kd}" />
-    <material>Gazebo/Black</material>
+    <!-- <material>Gazebo/Black</material> -->
   </gazebo>
   <!-- Wheel middle right -->
@@ -216,5 +208,5 @@
        <mesh filename="file://$(find zeus_description)/STL/Z1-PRP-01-001.stl"/>
       </geometry>
-      <material name="black"/>
+      <!-- <material name="black"/> -->
     </visual>
     <collision>
@@ -250,14 +242,14 @@
     <kp value="${wheel_kp}" />
     <kd value="${wheel_kd}" />
-    <material>Gazebo/Black</material>
+    <!-- <material>Gazebo/Black</material> -->
   </gazebo>
   <!-- Wheel rear right -->
   <link name="right_rear_wheel">
     <visual>
-      <origin rpy="${deg90} 0 0" xyz="0 0 0"/>
+      <origin rpy="0 0 0" xyz="0 0 0"/>
       <geometry>
         <mesh filename="file://$(find zeus_description)/STL/Z1-PRP-01-001.stl"/>
       </geometry>
-      <material name="black"/>
+      <!-- <material name="black"/> -->
     </visual>
     <collision>
@@ -265,5 +257,5 @@
         <cylinder length="${wheel_width}" radius="${wheel_radius}"/>
       </geometry>
-      <origin rpy="${deg90} 0 0" xyz="0 0 0"/>
+      <origin rpy="0 0 0" xyz="0 0 0"/>
     </collision>
     <inertial>
@@ -275,6 +267,6 @@
     <parent link="rocker_right"/>
     <child link="right_rear_wheel"/>
-    <origin rpy="0 0 0" xyz="-0.6 -0.05 -0.35"/>
-    <axis xyz="0 1 0"/>
+    <origin rpy="${deg90} 0 0" xyz="-0.6 -0.05 -0.35"/>
+    <axis xyz="0 0 -1"/>
   </joint>
   <transmission name="right_rear_wheel_trans">
@@ -293,5 +285,5 @@
     <kp value="${wheel_kp}" />
     <kd value="${wheel_kd}" />
-    <material>Gazebo/Black</material>
+    <!-- <material>Gazebo/Black</material> -->
   </gazebo>
   <!-- Wheel front left -->
@@ -302,5 +294,5 @@
        <mesh filename="file://$(find zeus_description)/STL/Z1-PRP-01-001.stl"/>
       </geometry>
-      <material name="black"/>
+      <!-- <material name="black"/> -->
     </visual>
     <collision>
@@ -319,5 +311,5 @@
     <child link="left_front_wheel"/>
    <origin rpy="${deg90} 0 0" xyz="0 0.05 -0.45"/>
-    <axis xyz="0 0 -1"/>
+    <axis xyz="0 0 1"/>
   </joint>
   <transmission name="left_front_wheel_trans">
@@ -336,5 +328,5 @@
     <kp value="${wheel_kp}" />
     <kd value="${wheel_kd}" />
-    <material>Gazebo/Black</material>
+    <!-- <material>Gazebo/Black</material> -->
   </gazebo>
   <!-- Wheel middle left -->
@@ -345,5 +337,5 @@
        <mesh filename="file://$(find zeus_description)/STL/Z1-PRP-01-001.stl"/>
       </geometry>
-      <material name="black"/>
+      <!-- <material name="black"/> -->
     </visual>
     <collision>
@@ -362,5 +354,5 @@
     <child link="left_middle_wheel"/>
     <origin rpy="${deg90} 0 0" xyz="-0.45 0.05 -0.05"/>
-    <axis xyz="0 0 -1"/>
+    <axis xyz="0 0 1"/>
   </joint>
   <transmission name="left_middle_wheel_trans">
@@ -379,14 +371,14 @@
     <kp value="${wheel_kp}" />
     <kd value="${wheel_kd}" />
-    <material>Gazebo/Black</material>
+    <!-- <material>Gazebo/Black</material> -->
   </gazebo>
   <!-- Wheel rear left -->
   <link name="left_rear_wheel">
     <visual>
-      <origin rpy="${deg90} 0 0" xyz="0 0 0"/>
+      <origin rpy="0 0 0" xyz="0 0 0"/>
       <geometry>
         <mesh filename="file://$(find zeus_description)/STL/Z1-PRP-01-001.stl"/>
       </geometry>
-      <material name="black"/>
+      <!-- <material name="black"/> -->
     </visual>
     <collision>
@@ -394,5 +386,5 @@
        <cylinder length="${wheel_width}" radius="${wheel_radius}"/>
       </geometry>
-      <origin rpy="${deg90} 0 0" xyz="0 0 0"/>
+      <origin rpy="0 0 0" xyz="0 0 0"/>
     </collision>
     <inertial>
@@ -404,6 +396,6 @@
     <parent link="rocker_left"/>
     <child link="left_rear_wheel"/>
-    <origin rpy="0 0 0" xyz="-0.6 0.05 -0.35"/>
-    <axis xyz="0 1 0"/>
+    <origin rpy="${deg90} 0 0" xyz="-0.6 0.05 -0.35"/>
+    <axis xyz="0 0 -1"/>
   </joint>
   <transmission name="left_rear_wheel_trans">
@@ -422,5 +414,5 @@
     <kp value="${wheel_kp}" />
     <kd value="${wheel_kd}" />
-    <material>Gazebo/Black</material>
+    <!-- <material>Gazebo/Black</material> -->
   </gazebo>
   <!-- IMU link -->

Commit message: Removed arm from simulation

File: zeus_description/urdf/zeus.urdf.xacro (robot description, xacro)
@@ -22,7 +22,7 @@
     <visual>
       <geometry>
-        <mesh filename="file://$(find zeus_description)/STL/Z1.stl"/>
-      </geometry>
-      <origin rpy="${deg90} 0 0" xyz="0 0 0"/>
+        <mesh filename="file://$(find zeus_description)/STL/chassis.stl"/>
+      </geometry>
+      <origin rpy="0 0 0" xyz="0 0 0"/>
     </visual>
     <collision>
@@ -32,8 +32,4 @@
       <origin rpy="0 0 0" xyz="0 0 0"/>
     </collision>
-    <inertial>
-      <mass value="${frame_mass}"/>
-      <inertia ixx="4" ixy="0.0" ixz="0.0" iyy="4" iyz="0.0" izz="4"/>
-    </inertial>
   </link>
   <gazebo reference="base_link">
@@ -56,5 +52,5 @@
     <parent link="base_link"/>
     <child link="rocker_right"/>
-    <origin rpy="0 -0.2 0" xyz="-0.3 -0.3 -0.4"/>
+    <origin rpy="0 -0.2 0" xyz="0 -0.3 0.05"/>
     <limit  lower="${-deg45}" upper="${deg45}" effort="100000.0" velocity="10.0"/>
     <axis xyz="0 1 0"/>
@@ -116,5 +112,5 @@
     <parent link="base_link"/>
     <child link="rocker_left"/>
-    <origin rpy="0 -0.2 0" xyz="-0.3 0.3 -0.4"/>
+    <origin rpy="0 -0.2 0" xyz="0 0.3 0.05"/>
     <limit  lower="${-deg45}" upper="${deg45}" effort="100000.0" velocity="10.0"/>
     <axis xyz="0 1 0"/>

Commit message: Added launch file for the base controller, Revert to simple simulation

File: zeus_description/urdf/zeus.urdf.xacro (robot description, xacro)
@@ -18,6 +18,7 @@
   <xacro:property name="wheel_kp" value="10000000.0" />
   <xacro:property name="wheel_kd" value="1" />
+  <link name="base_link" />
   <!-- Frame -->
-  <link name="base_link">
+  <link name="frame_link">
     <visual>
       <geometry>
@@ -32,6 +33,15 @@
       <origin rpy="0 0 0" xyz="0 0 0"/>
     </collision>
-  </link>
-  <gazebo reference="base_link">
+    <inertial>
+      <mass value="${frame_mass}"/>
+      <inertia ixx="4" ixy="0.0" ixz="0.0" iyy="4" iyz="0.0" izz="4"/>
+    </inertial>
+  </link>
+  <joint name="frame_joint" type="fixed">
+    <parent link="base_link" />
+    <child link="frame_link" />
+    <origin rpy="0 0 0" xyz="0 0 0"/>
+  </joint>
+  <gazebo reference="frame_link">
     <!-- <material>Gazebo/DarkGray</material> -->
   </gazebo>
@@ -50,5 +60,5 @@
   </link>
   <joint name="rocker_right_joint" type="revolute">
-    <parent link="base_link"/>
+    <parent link="frame_link"/>
     <child link="rocker_right"/>
     <origin rpy="0 -0.2 0" xyz="0 -0.3 0.05"/>
@@ -110,5 +120,5 @@
   </link>
   <joint name="rocker_left_joint" type="revolute">
-    <parent link="base_link"/>
+    <parent link="frame_link"/>
     <child link="rocker_left"/>
     <origin rpy="0 -0.2 0" xyz="0 0.3 0.05"/>
@@ -416,5 +426,5 @@
   <joint name="imu_joint" type="fixed">
     <origin xyz="0 0 0" rpy="0 0 0" />
-    <parent link="base_link" />
+    <parent link="frame_link" />
     <child link="imu_link" />
   </joint>
@@ -422,9 +432,9 @@
   </gazebo>
    <!-- Camera -->
-  <xacro:camera_sensor name="camera1" parent="base_link" hfov="1.3962634" image_width="800" image_height="600"  >
+  <xacro:camera_sensor name="camera1" parent="frame_link" hfov="1.3962634" image_width="800" image_height="600"  >
     <origin xyz="0.1 0 0" rpy="0 0 0" />
   </xacro:camera_sensor>
   <!-- Intel RealSense d435 -->
-  <xacro:realsense_d435_sensor name="d435" parent="base_link" >
+  <xacro:realsense_d435_sensor name="d435" parent="frame_link" >
     <origin xyz="0 0 0.5" rpy="0 0 0" />
   </xacro:realsense_d435_sensor>
@@ -440,5 +450,5 @@
       <robotNamespace>$(arg robot_namespace)</robotNamespace>
       <updateRate>50</updateRate>
-      <bodyName>base_link</bodyName>
+      <bodyName>frame_link</bodyName>
       <topicName>/imu/data</topicName>
       <accelDrift>0.005 0.005 0.005</accelDrift>
@@ -454,6 +464,6 @@
       <robotNamespace>$(arg robot_namespace)</robotNamespace>
       <updateRate>1</updateRate>
-      <bodyName>base_link</bodyName>
-      <frameId>base_link</frameId>
+      <bodyName>frame_link</bodyName>
+      <frameId>frame_link</frameId>
       <topicName>/fix</topicName>
       <velocityTopicName>navsat/vel</velocityTopicName>

Commit message: Options to load simple or complex simulation, fixed left rear wheel turning in wrong direction, added world with zero gravity to test robot without touching the ground

File: zeus_description/urdf/zeus.urdf.xacro (robot description, xacro)
@@ -403,5 +403,5 @@
     <child link="left_rear_wheel"/>
     <origin rpy="${deg90} 0 0" xyz="-0.6 0.05 -0.35"/>
-    <axis xyz="0 0 -1"/>
+    <axis xyz="0 0 1"/>
   </joint>
   <transmission name="left_rear_wheel_trans">
