Commit message: Include heartbeat in simulation launch; increased yaw tolerance for move_base

File: zeus_description/urdf/simple.urdf.xacro (robot description, xacro)
@@ -120,4 +120,8 @@
     <origin xyz="${base_x_size/2+0.01} 0 0" rpy="0 0 0" />
   </xacro:camera_sensor>
+  <!-- Zed depth camera -->
+  <!-- <xacro:zed_depth_cam name="zed" parent="base_link" >
+    <origin xyz="0 0 0.5" rpy="0 0 0" />
+  </xacro:zed_depth_cam> -->
   <!-- gazebo plugins -->
   <gazebo>
@@ -164,10 +168,10 @@
       <topicName>/fix</topicName>
       <velocityTopicName>navsat/vel</velocityTopicName>
-      <referenceLatitude>45.378395</referenceLatitude>
-      <referenceLongitude>-71.926644</referenceLongitude>
+      <referenceLatitude>45.3772267</referenceLatitude>
+      <referenceLongitude>-71.9277420</referenceLongitude>
       <referenceHeading>90</referenceHeading>
       <referenceAltitude>0</referenceAltitude>
       <drift>0.05 0.05 0.05</drift>
-      <gaussianNoise>1 1 1</gaussianNoise>
+      <gaussianNoise>0.1 0.1 0.1</gaussianNoise>
     </plugin>
   </gazebo>

Commit message: Zed urdf

File: zeus_description/urdf/simple.urdf.xacro (robot description, xacro)
@@ -2,5 +2,5 @@
 <robot name="simple" xmlns:xacro="http://ros.org/wiki/xacro">
   <xacro:include filename="$(find zeus_description)/urdf/accessories/camera.urdf.xacro"/>
-  <xacro:include filename="$(find zeus_description)/urdf/accessories/zed.urdf.xacro"/>
+  <xacro:include filename="$(find zed_wrapper)/urdf/zed_macro.urdf.xacro" />
   <xacro:arg name="robot_namespace" default="/" />
   <!-- Base size -->
@@ -121,7 +121,7 @@
   </xacro:camera_sensor>
   <!-- Zed depth camera -->
-  <!-- <xacro:zed_depth_cam name="zed" parent="base_link" >
-    <origin xyz="0 0 0.5" rpy="0 0 0" />
-  </xacro:zed_depth_cam> -->
+  <xacro:zed_camera name="zed" model="zed" parent="base_link">
+    <origin xyz="0 0 0" rpy="0 0 0" />
+  </xacro:zed_camera>
   <!-- gazebo plugins -->
   <gazebo>

File: zeus_description/urdf/zeus.urdf.xacro (robot description, xacro)
@@ -2,5 +2,5 @@
 <robot xmlns:xacro="http://www.ros.org/wiki/xacro" name="zeus">
   <xacro:include filename="$(find zeus_description)/urdf/accessories/camera.urdf.xacro"/>
-  <xacro:include filename="$(find zeus_description)/urdf/accessories/zed.urdf.xacro" />
+  <xacro:include filename="$(find zed_wrapper)/urdf/zed_macro.urdf.xacro" />
   <xacro:property name="deg90" value="1.57075" />
   <xacro:property name="deg45" value="0.7854" />
@@ -435,8 +435,8 @@
     <origin xyz="0.1 0 0" rpy="0 0 0" />
   </xacro:camera_sensor>
-  <!-- Intel RealSense d435 -->
-  <xacro:realsense_d435_sensor name="d435" parent="frame_link" >
-    <origin xyz="0 0 0.5" rpy="0 0 0" />
-  </xacro:realsense_d435_sensor>
+  <!-- Zed depth camera -->
+  <xacro:zed_camera name="zed" model="zed" parent="base_link">
+    <origin xyz="0 0 0" rpy="0 0 0" />
+  </xacro:zed_camera>
   <!-- Controllers -->
   <gazebo>

Commit message: Autonomous nav (#33)
* led_controller in autonomous_navigation.launch; SPI permissions on boot for LEDs

* Updated dependencies list

* Fixed multimaster not always finding other hosts

* Installations to make ROS melodic compatible with python3

* FIxed typo in repos list

* Fixed readme formating error

* typo and added missing multimaster instructions

* Fixed typo in installation script

* Upstart launch files and fisheye camera launch file

* Added tcp_repeater to repos list

* Added steve_science to repos list

* Increased fisheye camera resolution

* Removed base odom from EKF

* Changed branch for differential_drive

* Updated zed-ros-wrapper to 3.7

* Zed urdf

* zed: removed publish odom tf

* Moved tcp_publisher include to gps.launch

* Changed gps origin

* Changed diff drive rotation coefficient, changed gps frame_id and added nmea_navsat_driver to repos list

* Changed i2c_imu to rtimulib_ros package

* Using gps_heading for orientation, removed led_controller from autonomous_navigation launch file

* Coordinate visualizer for mapviz

* Moved instructions to wiki

* Correct imu frame name and fixed logic issue with base_controller launch

* imu launch file

* Fixed typo

* Changed IMU config

* Changed ekf to use zed odom

* Turned off rgbd_odometry

* addeed backcam

* Fixed bad global ekf config

* Standalone mapviz launch file

* Use gnss_to_map package, add dependencies, turned off obstacles detection

* Updated dependencies

* Removed navsat_transform_node from control launch file

Co-authored-by: Loic Boileau <boil3205@usherbrooke.ca>

File: zeus_description/urdf/simple.urdf.xacro (robot description, xacro)
@@ -2,5 +2,5 @@
 <robot name="simple" xmlns:xacro="http://ros.org/wiki/xacro">
   <xacro:include filename="$(find zeus_description)/urdf/accessories/camera.urdf.xacro"/>
-  <xacro:include filename="$(find zeus_description)/urdf/accessories/zed.urdf.xacro"/>
+  <xacro:include filename="$(find zed_wrapper)/urdf/zed_macro.urdf.xacro" />
   <xacro:arg name="robot_namespace" default="/" />
   <!-- Base size -->
@@ -121,7 +121,7 @@
   </xacro:camera_sensor>
   <!-- Zed depth camera -->
-  <!-- <xacro:zed_depth_cam name="zed" parent="base_link" >
-    <origin xyz="0 0 0.5" rpy="0 0 0" />
-  </xacro:zed_depth_cam> -->
+  <xacro:zed_camera name="zed" model="zed" parent="base_link">
+    <origin xyz="0 0 0" rpy="0 0 0" />
+  </xacro:zed_camera>
   <!-- gazebo plugins -->
   <gazebo>
@@ -168,6 +168,6 @@
       <topicName>/fix</topicName>
       <velocityTopicName>navsat/vel</velocityTopicName>
-      <referenceLatitude>45.3772267</referenceLatitude>
-      <referenceLongitude>-71.9277420</referenceLongitude>
+      <referenceLatitude>45.2961394</referenceLatitude>
+      <referenceLongitude>-71.9630744</referenceLongitude>
       <referenceHeading>90</referenceHeading>
       <referenceAltitude>0</referenceAltitude>
