Commit message: fixurdf

File: zeus_description/urdf/accessories/zed.urdf.xacro (robot description, xacro)
@@ -10,5 +10,5 @@
   <xacro:arg name="cam_pitch"     default="0.0" />
   <xacro:arg name="cam_yaw"       default="0.0" />
-  <xacro:include filename="$(find zed_wrapper)/urdf/zed_macro.urdf.xacro" />
+  <xacro:include filename="$(find zed_wrapper)/urdf/zed_descr.urdf.xacro" />
   <xacro:macro name="zed_depth_cam" params="parent *origin name" >
     <xacro:zed_depth_cam name="$(arg camera_name)" model="$(arg camera_model)" parent="$(arg base_frame)">

File: zeus_description/urdf/simple.urdf.xacro (robot description, xacro)
@@ -2,5 +2,9 @@
 <robot name="simple" xmlns:xacro="http://ros.org/wiki/xacro">
   <xacro:include filename="$(find zeus_description)/urdf/accessories/camera.urdf.xacro"/>
-  <xacro:include filename="$(find zeus_description)/urdf/accessories/zed.urdf.xacro" />
+  <xacro:include filename="$(find zeus_description)/urdf/accessories/zed.urdf.xacro">
+    <arg name="cam_pos_x" value="0"/>
+    <arg name="cam_pos_y" value="0"/>
+    <arg name="cam_pos_z" value="0.5"/>
+  </xacro:include>
   <xacro:arg name="robot_namespace" default="/" />
   <!-- Base size -->
@@ -120,8 +124,4 @@
     <origin xyz="${base_x_size/2+0.01} 0 0" rpy="0 0 0" />
   </xacro:camera_sensor>
-  <!-- Zed depth camera -->
-  <xacro:zed_depth_cam name="zed" parent="base_link" >
-    <origin xyz="0 0 0.5" rpy="0 0 0" />
-  </xacro:zed_depth_cam>
   <!-- gazebo plugins -->
   <gazebo>

Commit message: fix ZE BUG

File: zeus_description/urdf/accessories/zed.urdf.xacro (robot description, xacro)
@@ -10,9 +10,6 @@
   <xacro:arg name="cam_pitch"     default="0.0" />
   <xacro:arg name="cam_yaw"       default="0.0" />
-  <xacro:include filename="$(find zed_wrapper)/urdf/zed_descr.urdf.xacro" />
-  <xacro:macro name="zed_depth_cam" params="parent *origin name" >
-    <xacro:zed_depth_cam name="$(arg camera_name)" model="$(arg camera_model)" parent="$(arg base_frame)">
-      <origin xyz="$(arg cam_pos_x) $(arg cam_pos_y) $(arg cam_pos_z)" rpy="$(arg cam_roll) $(arg cam_pitch) $(arg cam_yaw)" />
-    </xacro:zed_depth_cam>
+  <xacro:macro name="zed_depth_cam" params="parent *origin name node_name" >
+    <xacro:include filename="$(find zed_wrapper)/urdf/zed_descr.urdf.xacro" />
     <gazebo reference="${name}_base_link">
       <sensor name="camera" type="depth">
@@ -37,9 +34,9 @@
             <updateRate>0.0</updateRate>
             <cameraName>${name}</cameraName>
-            <imageTopicName>/zed_node/rgb/image_rect_color</imageTopicName>
-            <cameraInfoTopicName>/zed_node/rgb/camera_info</cameraInfoTopicName>
-            <depthImageTopicName>/zed_node/depth/depth_registered</depthImageTopicName>
-            <depthImageCameraInfoTopicName>/zed_node/depth/camera_info</depthImageCameraInfoTopicName>
-            <pointCloudTopicName>/zed_node/point_cloud/cloud_registered</pointCloudTopicName>
+            <imageTopicName>/${node_name}/rgb/image_rect_color</imageTopicName>
+            <cameraInfoTopicName>/${node_name}/rgb/camera_info</cameraInfoTopicName>
+            <depthImageTopicName>/${node_name}/depth/depth_registered</depthImageTopicName>
+            <depthImageCameraInfoTopicName>/${node_name}/depth/camera_info</depthImageCameraInfoTopicName>
+            <pointCloudTopicName>/${node_name}/point_cloud/cloud_registered</pointCloudTopicName>
             <frameName>${name}_left_camera_optical_frame</frameName>
             <pointCloudCutoff>0.4</pointCloudCutoff>

File: zeus_description/urdf/simple.urdf.xacro (robot description, xacro)
@@ -2,9 +2,5 @@
 <robot name="simple" xmlns:xacro="http://ros.org/wiki/xacro">
   <xacro:include filename="$(find zeus_description)/urdf/accessories/camera.urdf.xacro"/>
-  <xacro:include filename="$(find zeus_description)/urdf/accessories/zed.urdf.xacro">
-    <arg name="cam_pos_x" value="0"/>
-    <arg name="cam_pos_y" value="0"/>
-    <arg name="cam_pos_z" value="0.5"/>
-  </xacro:include>
+  <xacro:include filename="$(find zeus_description)/urdf/accessories/zed.urdf.xacro"/>
   <xacro:arg name="robot_namespace" default="/" />
   <!-- Base size -->

Commit message: Fix simple.urdf (#32)
* fix wrong xacro name for zed

* returned to old name

* typo

* fixurdf

* fix ZE BUG

Co-authored-by: Loic Boileau <boil3205@usherbrooke.ca>

File: zeus_description/urdf/accessories/zed.urdf.xacro (robot description, xacro)
@@ -10,9 +10,6 @@
   <xacro:arg name="cam_pitch"     default="0.0" />
   <xacro:arg name="cam_yaw"       default="0.0" />
-  <xacro:include filename="$(find zed_wrapper)/urdf/zed_macro.urdf.xacro" />
-  <xacro:macro name="zed_depth_cam" params="parent *origin name" >
-    <xacro:zed_camera name="$(arg camera_name)" model="$(arg camera_model)" parent="$(arg base_frame)">
-      <origin xyz="$(arg cam_pos_x) $(arg cam_pos_y) $(arg cam_pos_z)" rpy="$(arg cam_roll) $(arg cam_pitch) $(arg cam_yaw)" />
-    </xacro:zed_camera>
+  <xacro:macro name="zed_depth_cam" params="parent *origin name node_name" >
+    <xacro:include filename="$(find zed_wrapper)/urdf/zed_descr.urdf.xacro" />
     <gazebo reference="${name}_base_link">
       <sensor name="camera" type="depth">
@@ -37,9 +34,9 @@
             <updateRate>0.0</updateRate>
             <cameraName>${name}</cameraName>
-            <imageTopicName>/zed_node/rgb/image_rect_color</imageTopicName>
-            <cameraInfoTopicName>/zed_node/rgb/camera_info</cameraInfoTopicName>
-            <depthImageTopicName>/zed_node/depth/depth_registered</depthImageTopicName>
-            <depthImageCameraInfoTopicName>/zed_node/depth/camera_info</depthImageCameraInfoTopicName>
-            <pointCloudTopicName>/zed_node/point_cloud/cloud_registered</pointCloudTopicName>
+            <imageTopicName>/${node_name}/rgb/image_rect_color</imageTopicName>
+            <cameraInfoTopicName>/${node_name}/rgb/camera_info</cameraInfoTopicName>
+            <depthImageTopicName>/${node_name}/depth/depth_registered</depthImageTopicName>
+            <depthImageCameraInfoTopicName>/${node_name}/depth/camera_info</depthImageCameraInfoTopicName>
+            <pointCloudTopicName>/${node_name}/point_cloud/cloud_registered</pointCloudTopicName>
             <frameName>${name}_left_camera_optical_frame</frameName>
             <pointCloudCutoff>0.4</pointCloudCutoff>

File: zeus_description/urdf/simple.urdf.xacro (robot description, xacro)
@@ -2,5 +2,5 @@
 <robot name="simple" xmlns:xacro="http://ros.org/wiki/xacro">
   <xacro:include filename="$(find zeus_description)/urdf/accessories/camera.urdf.xacro"/>
-  <xacro:include filename="$(find zeus_description)/urdf/accessories/zed.urdf.xacro" />
+  <xacro:include filename="$(find zeus_description)/urdf/accessories/zed.urdf.xacro"/>
   <xacro:arg name="robot_namespace" default="/" />
   <!-- Base size -->
@@ -120,8 +120,4 @@
     <origin xyz="${base_x_size/2+0.01} 0 0" rpy="0 0 0" />
   </xacro:camera_sensor>
-  <!-- Zed depth camera -->
-  <xacro:zed_depth_cam name="zed" parent="base_link" >
-    <origin xyz="0 0 0.5" rpy="0 0 0" />
-  </xacro:zed_depth_cam>
   <!-- gazebo plugins -->
   <gazebo>
